Commit message: Added first MoveIt config for IRB1300_11_90

File: abb_irb1300_support/urdf/irb1300_11_90_macro.xacro (robot description, xacro)
@@ -141,5 +141,5 @@
         </joint>
         <joint type="revolute" name="${prefix}joint_5">
-            <origin xyz="0.295574 0.0119 0" rpy="0 0 0"/>
+            <origin xyz="0.295574 0 0" rpy="0 0 0"/>
             <axis xyz="0 1 0"/>
             <parent link="${prefix}link_4"/>
@@ -150,5 +150,5 @@
         </joint>
         <joint type="revolute" name="${prefix}joint_6">
-            <origin xyz="0.084 -0.0119 0" rpy="0 0 0"/>
+            <origin xyz="0.084 0 0" rpy="0 0 0"/>
             <axis xyz="1 0 0"/>
             <parent link="${prefix}link_5"/>

Commit message: Changed Meshes to Collada

File: abb_irb1300_support/urdf/irb1300_11_90_macro.xacro (robot description, xacro)
@@ -13,7 +13,6 @@
             <visual name="visual">
                 <geometry>
-                    <mesh filename="package://abb_irb1300_support/meshes/irb1300_11_90/visual/base_link.stl" />
+                    <mesh filename="package://abb_irb1300_support/meshes/irb1300_11_90/visual/base_link.dae" />
                 </geometry>
-                <xacro:material_abb_graphite_white/>
             </visual>
         </link>
@@ -27,7 +26,6 @@
             <visual name="visual">
                 <geometry>
-                    <mesh filename="package://abb_irb1300_support/meshes/irb1300_11_90/visual/link_1.stl" />
+                    <mesh filename="package://abb_irb1300_support/meshes/irb1300_11_90/visual/link_1.dae" />
                 </geometry>
-                <xacro:material_abb_graphite_white/>
             </visual>
         </link>
@@ -41,7 +39,6 @@
             <visual name="visual">
                 <geometry>
-                    <mesh filename="package://abb_irb1300_support/meshes/irb1300_11_90/visual/link_2.stl" />
+                    <mesh filename="package://abb_irb1300_support/meshes/irb1300_11_90/visual/link_2.dae" />
                 </geometry>
-                <xacro:material_abb_graphite_white/>
             </visual>
         </link>
@@ -55,7 +52,6 @@
             <visual name="visual">
                 <geometry>
-                    <mesh filename="package://abb_irb1300_support/meshes/irb1300_11_90/visual/link_3.stl" />
+                    <mesh filename="package://abb_irb1300_support/meshes/irb1300_11_90/visual/link_3.dae" />
                 </geometry>
-                <xacro:material_abb_graphite_white/>
             </visual>
         </link>
@@ -69,7 +65,6 @@
             <visual name="visual">
                 <geometry>
-                    <mesh filename="package://abb_irb1300_support/meshes/irb1300_11_90/visual/link_4.stl" />
+                    <mesh filename="package://abb_irb1300_support/meshes/irb1300_11_90/visual/link_4.dae" />
                 </geometry>
-                <xacro:material_abb_graphite_white/>
             </visual>
         </link>
@@ -83,7 +78,6 @@
             <visual name="visual">
                 <geometry>
-                    <mesh filename="package://abb_irb1300_support/meshes/irb1300_11_90/visual/link_5.stl" />
+                    <mesh filename="package://abb_irb1300_support/meshes/irb1300_11_90/visual/link_5.dae" />
                 </geometry>
-                <xacro:material_abb_graphite_white/>
             </visual>
         </link>
@@ -97,7 +91,6 @@
             <visual name="visual">
                 <geometry>
-                    <mesh filename="package://abb_irb1300_support/meshes/irb1300_11_90/visual/link_6.stl" />
+                    <mesh filename="package://abb_irb1300_support/meshes/irb1300_11_90/visual/link_6.dae" />
                 </geometry>
-                <xacro:material_abb_graphite_white/>
             </visual>
         </link>
